File: Akashi-13.kicad_pcb (KiCad board)
At the start: 2 copper layers, 67.3 x 91.4 mm, 38 parts, among them J1 Conn_02x35_Odd_Even, J2 Conn_02x35_Odd_Even, J3 CONN12_011D01BNL_PUL, U1 LAN9220-ABZJ, U2 93AA46AT-IOT, X1 DFA-S15

Commit message: in the middle of routing
Parts:
- moved C16 2.06 mm to (130.2, 100.8)
- moved C17 1.95 mm to (134.2, 100.9)
Routing:
- net +3.3V: track 12.0 -> 14.4 mm
- net +1V8: track 20.6 -> 21.7 mm
Changed lines of the file:
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@@
   )
   (footprint "Capacitor_SMD:C_0603_1608Metric_Pad1.08x0.95mm_HandSolder" (layer "B.Cu")
-    (at 130.75 102.75 90)
+    (at 130.25 100.75 90)
     (descr "Capacitor SMD 0603 (1608 Metric), square (rectangular) end terminal, IPC_7351 nominal with elongated pad for handsoldering. (Body size source: IPC-SM-782 page 76, https://www.pcb-3d.com/wordpress/wp-content/uploads/ipc-sm-782a_amendment_1_and_2.pdf), generated with kicad-footprint-generator")
     (tags "capacitor handsolder")
@@
   )
   (footprint "Capacitor_SMD:C_0603_1608Metric_Pad1.08x0.95mm_HandSolder" (layer "B.Cu")
-    (at 133.75 102.75 90)
+    (at 134.25 100.8625 90)
     (descr "Capacitor SMD 0603 (1608 Metric), square (rectangular) end terminal, IPC_7351 nominal with elongated pad for handsoldering. (Body size source: IPC-SM-782 page 76, https://www.pcb-3d.com/wordpress/wp-content/uploads/ipc-sm-782a_amendment_1_and_2.pdf), generated with kicad-footprint-generator")
     (tags "capacitor handsolder")
@@
   (via (at 129.25 131) (size 0.6) (drill 0.2) (layers "F.Cu" "B.Cu") (net 72))
   (segment (start 127.95625 131) (end 129.25 131) (width 0.2) (layer "B.Cu") (net 72))
-  (segment (start 130.78 106.3225) (end 130.78 104.78) (width 0.25) (layer "F.Cu") (net 129))
-  (segment (start 133.78 106.3225) (end 133.78 104.78) (width 0.25) (layer "F.Cu") (net 129))
+  (segment (start 133.78 106.3225) (end 133.78 104.22) (width 0.25) (layer "F.Cu") (net 129))
+  (segment (start 133.78 104.22) (end 134.25 103.75) (width 0.25) (layer "F.Cu") (net 129))
   (segment (start 136.933058 113.566942) (end 137.5 114.133884) (width 0.25) (layer "F.Cu") (net 129))
-  (segment (start 130.78 104.78) (end 130.75 104.75) (width 0.25) (layer "F.Cu") (net 129))
-  (segment (start 133.75 104.75) (end 133.78 104.78) (width 0.25) (layer "F.Cu") (net 129))
   (segment (start 136.876116 113.51) (end 136.933058 113.566942) (width 0.25) (layer "F.Cu") (net 129))
   (segment (start 135.9675 113.51) (end 136.876116 113.51) (width 0.25) (layer "F.Cu") (net 129))
@@
   (segment (start 117.8875 115.8) (end 117.8875 114.6125) (width 0.25) (layer "F.Cu") (net 129))
   (segment (start 137.5 114.133884) (end 137.5 114.75) (width 0.25) (layer "F.Cu") (net 129))
+  (segment (start 130.75 104.25) (end 130.25 103.75) (width 0.25) (layer "F.Cu") (net 129))
   (segment (start 126.51 107.51) (end 126.5 107.5) (width 0.25) (layer "F.Cu") (net 129))
   (segment (start 130.28 115.72) (end 130.25 115.75) (width 0.25) (layer "F.Cu") (net 129))
   (segment (start 117.8875 114.6125) (end 118 114.5) (width 0.25) (layer "F.Cu") (net 129))
   (segment (start 135.28 114.78) (end 136.25 115.75) (width 0.25) (layer "F.Cu") (net 129))
+  (segment (start 130.78 106.3225) (end 130.78 104.28) (width 0.25) (layer "F.Cu") (net 129))
+  (segment (start 130.78 104.28) (end 130.75 104.25) (width 0.25) (layer "F.Cu") (net 129))
   (segment (start 135.28 114.1975) (end 135.28 114.78) (width 0.25) (layer "F.Cu") (net 129))
   (segment (start 128.0925 107.51) (end 126.51 107.51) (width 0.25) (layer "F.Cu") (net 129))
@@
   (via (at 137.5 114.75) (size 0.6) (drill 0.2) (layers "F.Cu" "B.Cu") (net 129))
   (via (at 136.25 115.75) (size 0.6) (drill 0.2) (layers "F.Cu" "B.Cu") (net 129))
-  (via (at 133.78 104.78) (size 0.6) (drill 0.2) (layers "F.Cu" "B.Cu") (net 129))
+  (via (at 134.25 103.75) (size 0.6) (drill 0.2) (layers "F.Cu" "B.Cu") (net 129))
   (via (at 130.25 115.75) (size 0.6) (drill 0.2) (layers "F.Cu" "B.Cu") (net 129))
-  (via (at 130.75 104.75) (size 0.6) (drill 0.2) (layers "F.Cu" "B.Cu") (net 129))
+  (via (at 130.25 103.75) (size 0.6) (drill 0.2) (layers "F.Cu" "B.Cu") (net 129))
   (segment (start 133.78 114.1975) (end 133.78 115.348745) (width 0.25) (layer "F.Cu") (net 130))
   (segment (start 133.78 115.348745) (end 134.200735 115.76948) (width 0.25) (layer "F.Cu") (net 130))
-  (segment (start 135.9675 113.01) (end 137.24 113.01) (width 0.25) (layer "F.Cu") (net 130))
+  (segment (start 137.24 113.01) (end 135.9675 113.01) (width 0.25) (layer "F.Cu") (net 130))
+  (segment (start 137.75 113.5) (end 137.24 113.01) (width 0.25) (layer "F.Cu") (net 130))
   (segment (start 126.51 111.01) (end 126.5 111) (width 0.25) (layer "F.Cu") (net 130))
   (segment (start 128.0925 111.01) (end 126.51 111.01) (width 0.25) (layer "F.Cu") (net 130))
-  (segment (start 137.24 113.01) (end 137.25 113) (width 0.25) (layer "F.Cu") (net 130))
   (via (at 134.200735 115.76948) (size 0.6) (drill 0.2) (layers "F.Cu" "B.Cu") (net 130))
   (via (at 126.5 111) (size 0.6) (drill 0.2) (layers "F.Cu" "B.Cu") (net 130))
-  (via (at 137.25 113) (size 0.6) (drill 0.2) (layers "F.Cu" "B.Cu") (net 130))
-  (segment (start 137.25 113) (end 134.25 113) (width 0.25) (layer "B.Cu") (net 130))
+  (via (at 137.75 113.5) (size 0.6) (drill 0.2) (layers "F.Cu" "B.Cu") (net 130))
+  (segment (start 138.8875 113) (end 138.25 113) (width 0.25) (layer "B.Cu") (net 130))
   (segment (start 129.5 111) (end 126.5 111) (width 0.25) (layer "B.Cu") (net 130))
   (segment (start 134.200735 115.76948) (end 134.200735 113.049265) (width 0.25) (layer "B.Cu") (net 130))
   (segment (start 134.25 113) (end 131.5 113) (width 0.25) (layer "B.Cu") (net 130))
-  (segment (start 137.25 113) (end 138.8875 113) (width 0.25) (layer "B.Cu") (net 130))
   (segment (start 134.200735 113.049265) (end 134.25 113) (width 0.25) (layer "B.Cu") (net 130))
+  (segment (start 137.25 113) (end 137.75 113.5) (width 0.25) (layer "B.Cu") (net 130))
+  (segment (start 134.25 113) (end 137.25 113) (width 0.25) (layer "B.Cu") (net 130))
+  (segment (start 138.25 113) (end 137.75 113.5) (width 0.25) (layer "B.Cu") (net 130))
   (segment (start 131.5 113) (end 129.5 111) (width 0.25) (layer "B.Cu") (net 130))
   (segment (start 132.28 115.53) (end 132.5 115.75) (width 0.25) (layer "F.Cu") (net 139))

Commit message: Layout done.
Parts:
- moved C15 0.62 mm to (124.9, 107.5)
Routing:
- net GND: track 0.00 -> 119.5 mm, vias 0 -> 11
- net +3.3V: track 14.4 -> 121.6 mm, vias 7 -> 18
- net /D15: track 0.00 -> 90.2 mm
- net /D14: track 0.00 -> 76.2 mm
- net /D4: track 0.00 -> 75.8 mm, vias 0 -> 3
- net /A5: track 0.00 -> 75.6 mm, vias 0 -> 1
- net /A4: track 0.00 -> 72.2 mm, vias 0 -> 2
- net /D0: track 0.00 -> 70.9 mm, vias 0 -> 3
- net /nRESET: track 0.00 -> 64.1 mm, vias 0 -> 2
- net /D5: track 0.00 -> 63.7 mm, vias 0 -> 3
- net /D10: track 0.00 -> 61.9 mm, vias 0 -> 1
- net /D6: track 0.00 -> 60.8 mm, vias 0 -> 1
- net /D9: track 0.00 -> 58.3 mm, vias 0 -> 1
- net /D8: track 0.00 -> 57.2 mm, vias 0 -> 1
- net /D13: track 0.00 -> 55.6 mm, vias 0 -> 3
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- added copper zone on In2.Cu, net +3.3V
- added copper zone on In1.Cu, net GND
- removed copper zone on F.Cu, net +3.3V
- removed copper zone on B.Cu, net GND
Other:
- copper layers 2 -> 4
