File: Akashi-13.kicad_pcb (KiCad board)
At the start: 4 copper layers, 67.3 x 91.4 mm, 38 parts, among them J1 Conn_02x35_Odd_Even, J2 Conn_02x35_Odd_Even, J3 CONN12_011D01BNL_PUL, U1 LAN9220-ABZJ, U2 93AA46AT-IOT, X1 DFA-S15

Commit message: Add comment on the board.
JB1
LEDs
Other:
- board text added: "(C) Seiichi Horie, 2023 https://github.com/suikan4github/Akashi-13"
- board text added: "Akashi-13"
- board text added: "Ethernet board for Nucleo 144"
- board text added: "FULL DUPLEX"
- board text added: "JB1 : AUTO MDIX OPEN => ENABLE SHORT => DISABLE"
- board text added: "LINK ACT"
- board text added: "SPEED 100"
Changed lines of the file:
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@@
   (gr_line (start 151.13 77.47) (end 111.76 77.47)
     (stroke (width 0.1) (type default)) (layer "Edge.Cuts"))
+  (gr_text "(C) Seiichi Horie, 2023\nhttps://github.com/suikan4github/Akashi-13" (at 148.59 90.17) (layer "F.SilkS")
+    (effects (font (size 1 1) (thickness 0.15)) (justify left bottom mirror))
+  )
+  (gr_text "JB1  : AUTO MDIX\n    OPEN  => ENABLE\n    SHORT => DISABLE \n" (at 121.92 129.54) (layer "F.SilkS")
+    (effects (font (size 1 1) (thickness 0.15)) (justify left bottom))
+  )
+  (gr_text "Akashi-13" (at 112.75 84.75) (layer "F.SilkS")
+    (effects (font (size 2 2) (thickness 0.3)) (justify left bottom))
+  )
+  (gr_text "SPEED 100" (at 140.97 153.67) (layer "F.SilkS")
+    (effects (font (size 1 1) (thickness 0.15)) (justify left bottom))
+  )
+  (gr_text "Ethernet board for Nucleo 144" (at 112.5 87.25) (layer "F.SilkS")
+    (effects (font (size 1 1) (thickness 0.15)) (justify left bottom))
+  )
+  (gr_text "LINK ACT" (at 115.57 153.67) (layer "F.SilkS")
+    (effects (font (size 1 1) (thickness 0.15)) (justify left bottom))
+  )
+  (gr_text "FULL DUPLEX" (at 144.78 151.13) (layer "F.SilkS")
+    (effects (font (size 1 1) (thickness 0.15)) (justify left bottom))
+  )
   (dimension (type aligned) (layer "Cmts.User")
     (pts (xy 100.33 132.08) (xy 132.08 132.08))
     (height 35.56)
-    (gr_text "1250.0000 mils" (at 116.205 166.49) (layer "Cmts.User")
+    (gr_text "31.7500 mm" (at 116.205 166.49) (layer "Cmts.User")
       (effects (font (size 1 1) (thickness 0.15)))
     )
@@
     (pts (xy 100.33 151.13) (xy 163.83 151.13))
     (height 11.43)
-    (gr_text "2500.0000 mils" (at 132.08 160.76) (layer "Cmts.User")
+    (gr_text "63.5000 mm" (at 132.08 160.76) (layer "Cmts.User")
       (effects (font (size 1.5 1.5) (thickness 0.3)))
     )
@@
     (style (thickness 0.2) (arrow_length 1.27) (text_position_mode 0) (extension_height 0.58642) (extension_offset 0.5) keep_text_aligned)
   )
+  (dimension (type aligned) (layer "Cmts.User")
+    (pts (xy 165.1 154.94) (xy 165.1 63.5))
+    (height 4.15)
+    (gr_text "91.4400 mm" (at 168.1 109.22 90) (layer "Cmts.User")
+      (effects (font (size 1 1) (thickness 0.15)))
+    )
+    (format (prefix "") (suffix "") (units 3) (units_format 1) (precision 4))
+    (style (thickness 0.15) (arrow_length 1.27) (text_position_mode 0) (extension_height 0.58642) (extension_offset 0.5) keep_text_aligned)
+  )
   (segment (start 131.25 114.198) (end 131.25 114.1975) (width 0.25) (layer "F.Cu") (net 8))
